File: PCB/Occupancy PCB Final Rev B.brd (EAGLE design)
At the start: 74 x 60 mm, 10 parts

Commit message: Ovie's final edit to pins
Parts:
- moved XBEE 7.13 mm to (37.5, 15.5), turned to 0 degrees
- moved CO2 5.95 mm to (42.0, 42.6)
- moved PIR 5.08 mm to (38.0, 67.1)
- moved R4 4.60 mm to (38.5, 43.6)
- moved R1 4.10 mm to (38.5, 35.1)
- moved R2 4.10 mm to (38.5, 39.1)
Connections:
- removed net N$11: LAUNCHPAD.28, XBEE.18
- new net N$1: LAUNCHPAD.31, XBEE.18
Routing:
- net N$5: track 15.1 -> 65.4 mm
- net N$1: track 0.00 -> 39.5 mm
- net N$4: track 0.00 -> 36.6 mm
- net VCC: track 89.4 -> 111.7 mm
- net N$3: track 48.1 -> 67.2 mm
- net N$10: track 0.00 -> 11.4 mm
- net N$6: track 40.2 -> 45.8 mm, vias 0 -> 1
- net VDD: track 50.6 -> 52.6 mm
- net N$12: track 98.2 -> 100.1 mm
- net N$2: track 44.6 -> 45.7 mm
- net N$8: track 70.9 -> 71.9 mm
Other:
- board text added: "GND"
- board text added: "VCC"
- board text added: "VDD"
- board text removed: "A few more labels would be good, too. Remember: you might be soldering this when you're tired. Especially note the required orientation of the Tiva / Launchpad."
- board text removed: "How do you plan to hold the PIR sensor onto the board when it's upside down? If you need mount holes, you should add them."
- board text removed: "It looks like you've tied two SPI pins (MISO and MOSI) together -- why?"
- board text removed: "Try flipping the PIR module around and moving the DHT11 to the lower left of the BoosterPack. You could cut off 1/3 of the whole board. Fixed."
- board text removed: "Vertical clearance of each module? Could you make this more compact? (especially the 3-pin CO2 and 3-pin PIR modules)"
- board text removed: "You made ground planes but never attached them to GND. Fixed."
- board text removed: "You need to put a Vcc supply symbol on the schematic. It makes routing work a lot better."
- board text removed: "You've got a mixed 3V3 and 5V system. Make Vcc and Vdd. Worse, your I2C bus was getting 5V pumped into its 3V3 logic levels. Fixed."
